Commit message: running robot in gazebo

File: description/robot.urdf.xacro (robot description, xacro)
@@ -6,3 +6,6 @@
     <xacro:include filename="colors.xacro" />
     <xacro:include filename="sensors.xacro" />
+    <!--Gazebo-->
+    <xacro:include filename="/home/ran/robot_ws/src/captain-robot/description/gazebo/gazebo_colors.xacro" />
+        <xacro:include filename="/home/ran/robot_ws/src/captain-robot/description/gazebo/gazebo_control.xacro" />
 </robot>

File: description/robot_core.xacro (robot description, xacro)
@@ -2,5 +2,6 @@
 <robot xmlns:xacro="http://www.ros.org/wiki/xacro">
 <!--Base Link-->
-<link name="base_link">
+<link name = 'base_link'></link>
+<link name="chassis">
     <visual>
         <origin xyz="0 0 0.025" rpy="0 0 0"/>
@@ -20,3 +21,8 @@
     </xacro:inertial_cylinder>
 </link>
+<joint name="chassis_joint" type="fixed">
+    <parent link="base_link"/>
+    <child link="chassis"/>
+    <origin xyz="0 0 0" rpy="0 0 0"/>
+</joint>
 </robot>
