Commit message: fixes

File: description/gazebo_properties.xacro (robot description, xacro)
@@ -44,5 +44,5 @@
             <plugin name="laser_controller" filename="libgazebo_ros_ray_sensor.so">
                 <ros>
-                    <argument>~/out:=scan</argument>
+                    <argument>--ros-args --remap ~/out:=scan</argument>
                 </ros>
                 <output_type>sensor_msgs/LaserScan</output_type>

File: description/robot.urdf.xacro (robot description, xacro)
@@ -1,11 +1,15 @@
 <?xml version="1.0"?>
 <robot xmlns:xacro="http://www.ros.org/wiki/xacro"  name="robot">
+    <!--Design-->
     <xacro:include filename="inertial_macros.xacro" />
     <xacro:include filename="robot_core.xacro" />
     <xacro:include filename="wheels.xacro" />
     <xacro:include filename="colors.xacro" />
+    <!--Control-->
+    <xacro:include filename="ros2_control.xacro" />
+    <!--Sensors-->
     <xacro:include filename="sensors.xacro" />
     <!--Gazebo-->
-    <xacro:include filename="/gazebo/gazebo_properties.xacro" />
-    <xacro:include filename="/gazebo/gazebo_control.xacro" />
+    <xacro:include filename="gazebo_properties.xacro" />
+    <!-- <xacro:include filename="gazebo_control.xacro" /> -->
 </robot>

File: description/robot_core.xacro (robot description, xacro)
@@ -3,4 +3,12 @@
 <!--Base Link-->
 <link name = 'base_link'></link>
+<!--Base Footprint-->
+<link name = 'base_footprint'></link>
+<joint name="footprint_joint" type="fixed">
+    <parent link="base_link"/>
+    <child link="base_footprint"/>
+    <origin xyz="0 0 0" rpy="0 0 0"/>
+</joint>
+<!--Chassis-->
 <link name="chassis">
     <visual>
